File: PCB/Carga util/Carga_util_V2-k/Carga util.kicad_sch (KiCad schematic)
At the start: 37 parts, among them J1 CONN, J2 BG51, J3 DEBUG, J4 UART, Q1 NMOS, Q2 NMOS, SW1 Reset, U1 ATtiny85-20S, U2 LM1117DT-3.3

Commit message: Add lock files for autosave of schematic and PCB with user details
Parts:
- removed J3: DEBUG, Connector_PinHeader_1.27mm:PinHeader_1x04_P1.27mm_Vertical, symbol Connector:Conn_01x04_Socket
- removed J4: UART, Connector_PinHeader_1.27mm:PinHeader_1x04_P1.27mm_Vertical, symbol Connector:Conn_01x04_Socket
- removed TP5: Test_GND, symbol Connector:TestPoint_Probe
- added J1: UART, Connector_PinHeader_2.54mm:PinHeader_1x04_P2.54mm_Vertical, symbol Connector:Conn_01x04_Pin
- added J3: DEBUG, Connector_PinHeader_2.54mm:PinHeader_1x06_P2.54mm_Vertical, symbol Connector:Conn_01x06_Pin
- added J5, J6: Conn_01x02_Pin, Connector_PinHeader_2.54mm:PinHeader_1x02_P2.54mm_Vertical, symbol Connector:Conn_01x02_Pin
- added TP6: Test_GND, TestPoint:TestPoint_Pad_2.0x2.0mm, symbol Connector:TestPoint_Probe
- C6: renamed from C2; value 4.7u -> 4.7uF
- D1: renamed from D3; footprint (none) -> Diode_SMD:D_SMF
- F1: footprint (none) -> Fuse:Fuse_0805_2012Metric
- JP2, JP3: footprint (none) -> Jumper:SolderJumper-2_P1.3mm_Open_Pad1.0x1.5mm
- Q1, Q2: footprint (none) -> Package_TO_SOT_SMD:SOT-23
- R5: renamed from R10; footprint (none) -> Resistor_SMD:R_0805_2012Metric
- R6: renamed from R9; footprint (none) -> Resistor_SMD:R_0805_2012Metric
- R8: renamed from R11; footprint (none) -> Resistor_SMD:R_0805_2012Metric
- R9: renamed from R12; footprint (none) -> Resistor_SMD:R_0805_2012Metric
- TP1: footprint (none) -> TestPoint:TestPoint_Pad_2.0x2.0mm
- TP2: renamed from TP3; footprint (none) -> TestPoint:TestPoint_Pad_2.0x2.0mm
- TP4: renamed from TP2; footprint (none) -> TestPoint:TestPoint_Pad_2.0x2.0mm
- TP5: renamed from TP4; footprint (none) -> TestPoint:TestPoint_Pad_2.0x2.0mm
- renumbered C3 to C1, C4 to C2, C5 to C3, C6 to C4, C1 to C5, D1 to D2, D2 to D3, J1 to J2, J2 to J4, R3 to R1, R6 to R10, R1 to R2, R2 to R3, R5 to R7, U2 to U1, U1 to U2
Connections:
- net VCC is gone; now on net +3.3V: R4.1, U2.8 (VCC)
- net +3.3V: now also J1.2 (Pin_2), J3.6 (Pin_6)
- net +3.7V: no longer J2.1 (Pin_1)
- net GND: now also J1.1 (Pin_1), J3.5 (Pin_5), J5.2 (Pin_2), TP6.1
- net SCL: now also J3.1 (Pin_1)
- net SCL_HV: now also J6.2 (Pin_2)
- net SDA: now also J1.4 (Pin_4), J3.3 (Pin_3)
- net SDA_HV: now also J6.1 (Pin_1)
- net IN: now reaches F1.2, TP1.1
- net IN: now also J2.1 (Pin_1), J5.1 (Pin_1)
- net LED_Test renamed SS
- net SS: now also J3.4 (Pin_4); no longer JP1.2 (B), U2.3 (XTAL2/PB4)
- net MISO renamed DO
- net DO: now also J1.3 (Pin_3), J3.2 (Pin_2)
- net VCC_Filter renamed VDC_Filter
- new net: JP1.2 (B), U2.3 (XTAL2/PB4)
Other:
- moved on the sheet: D3, J2, J4, JP1, R10, R4, R7, SW1, TP1, TP4, TP5, U2
