File: PCB/Carga util/Carga_util_V2-k/_autosave-Carga util.kicad_pcb (KiCad board)
At the start: 2 copper layers, 57.5 x 53.5 mm, 42 parts, among them J1 UART, J2 CONN, J3 DEBUG, J4 BG51, J5 Conn_01x02_Pin, J6 Conn_01x02_Pin, Q1 NMOS, Q2 NMOS, SW1 Reset, U1 LM1117DT-3.3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

Commit message: Add lock files for autosave of schematic and PCB with user details
Parts:
- removed REF**: Arduino_UNO_R3_WithMountingHoles, Module:Arduino_UNO_R3_WithMountingHoles
- added ?: , , F.Cu at (178.4, 77.9)
- added ?: , , F.Cu at (127.6, 62.7)
- added ?: , , F.Cu at (178.5, 105.9)
- added ?: , , F.Cu at (126.4, 111.0)
- D2: footprint LED_SMD:LED_0603_1608Metric -> LED_SMD:LED_0805_2012Metric
- F1: footprint Fuse:Fuse_0805_2012Metric -> Fuse:Fuse_1206_3216Metric
- moved G*** 45.6 mm to (174.0, 99.0)
- moved +3.3V 8.20 mm to (164.3, 105.5)
- moved D1 8.20 mm to (139.1, 106.2)
- moved D3 8.20 mm to (145.9, 92.6)
- moved GND 8.20 mm to (155.8, 102.5)
- moved IN 8.20 mm to (155.8, 105.5)
- moved J1 8.20 mm to (147.8, 68.5)
- moved J2 8.20 mm to (144.3, 103.2)
- moved J3 8.20 mm to (147.8, 72.5)
- moved J4 8.20 mm to (158.3, 85.0)
- moved JP1 8.20 mm to (145.9, 88.2)
- moved JP3 8.20 mm to (155.9, 97.7)
- moved PP 8.20 mm to (166.3, 92.5)
- moved Q1 8.20 mm to (151.4, 95.3)
- moved R10 8.20 mm to (154.1, 82.4)
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- renumbered TP2 to +3.3V, TP6 to GND, TP1 to IN, TP5 to PP, TP4 to VCCF
Routing:
- net /IN: track 46.3 -> 38.1 mm
- net /SCK: track 43.2 -> 40.3 mm
- net /DI: track 48.5 -> 47.4 mm
- net /SDA_HV: track 46.4 -> 47.6 mm
- net /SCL_HV: track 41.3 -> 42.5 mm
- net (no net): vias 4 -> 0
Other:
- board size 57.5 x 53.5 mm -> 57.8 x 53.9 mm
- board text added: "+"
- board text added: "-"
- board text added: "PP"
