File: PCB/Carga util/Carga_util_V2- arduino/Carga util.kicad_pcb (KiCad board)
At the start: 2 copper layers, 57.8 x 53.9 mm, 45 parts, among them J1 UART, J2 CONN, J3 DEBUG, J4 BG51, J5 Conn_01x02_Pin, J6 Conn_01x02_Pin, Q1 NMOS, Q2 NMOS, SW1 Reset, U1 LM1117DT-3.3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

Commit message: nuevo pcb
Parts:
- removed the G*** at (184.5, 106.7)
- C1, C4: footprint Capacitor_Tantalum_SMD:CP_EIA-1608-08_AVX-J -> Capacitor_Tantalum_SMD:CP_EIA-2012-15_AVX-P
- D3: footprint LED_SMD:LED_0603_1608Metric -> LED_SMD:LED_0805_2012Metric
- J3: footprint Connector_PinHeader_2.54mm:PinHeader_1x06_P2.54mm_Vertical -> Connector_PinHeader_2.54mm:PinHeader_1x04_P2.54mm_Vertical
- SW1: footprint Button_Switch_SMD:SW_SPST_TL3342 -> Button_Switch_THT:SW_PUSH_6mm
- moved J4 11.7 mm to (169.8, 87.4), turned to -90 degrees
- moved R10 3.80 mm to (157.9, 82.5)
- moved PP 3.75 mm to (169.8, 94.0)
- moved VCCF 3.40 mm to (166.2, 93.9)
- moved SW1 3.19 mm to (136.9, 88.2)
- moved R1 3.16 mm to (147.4, 98.1), turned to 180 degrees
- moved D2 3.12 mm to (147.3, 95.9)
- moved R3 3.06 mm to (154.9, 82.5)
- moved R2 3.06 mm to (151.8, 82.4)
- moved G*** 1.76 mm to (173.4, 100.6)
- moved D3 1.66 mm to (147.4, 93.2)
- moved R7 1.56 mm to (147.4, 90.8)
- moved JP1 1.56 mm to (147.4, 88.4)
- moved U2 0.99 mm to (134.3, 74.7)
- moved C6 0.77 mm to (154.8, 78.7)
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Routing:
- net /VDC_Filter: track 24.7 -> 52.7 mm
- net /PP: track 43.9 -> 55.4 mm
- net /IN: track 38.1 -> 45.8 mm
- net Net-(JP1-B): track 23.2 -> 29.2 mm
- net /SS: track 62.0 -> 66.2 mm
- net /DI: track 47.4 -> 50.3 mm
- net /SCK: track 40.3 -> 42.7 mm
- net +3.3V: track 176.6 -> 175.0 mm
- net /SDA_HV: track 47.6 -> 49.1 mm
- net +3.7V: track 69.8 -> 70.6 mm
- net /DO: track 17.7 -> 17.0 mm
Other:
- board size 57.8 x 53.9 mm -> 57.8 x 54.2 mm
