File: PCB/Carga util/Carga_util_V2- arduino/Carga util.kicad_sch (KiCad schematic)
At the start: 39 parts, among them J1 UART, J2 CONN, J3 DEBUG, J4 BG51, J5 Conn_01x02_Pin, J6 Conn_01x02_Pin, Q1 NMOS, Q2 NMOS, SW1 Reset, U1 LM1117DT-3.3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

Commit message: nuevo pcb
Parts:
- J3: symbol Connector:Conn_01x06_Pin -> Connector:Conn_01x04_Pin
Connections:
- net +3.3V: no longer J3.6 (Pin_6)
- net GND: no longer J3.5 (Pin_5)
Changed lines of the file:
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@@
 	(wire
 		(pts
-			(xy 88.9 74.93) (xy 91.44 74.93)
-		)
-		(stroke
-			(width 0)
-			(type default)
-		)
-	)
-	(wire
-		(pts
 			(xy 76.2 82.55) (xy 95.25 82.55)
 		)
@@
 	(wire
 		(pts
-			(xy 91.44 74.93) (xy 91.44 77.47)
-		)
-		(stroke
-			(width 0)
-			(type default)
-		)
-	)
-	(wire
-		(pts
 			(xy 130.81 95.25) (xy 142.24 95.25)
 		)
@@
 	(wire
 		(pts
-			(xy 92.71 74.93) (xy 95.25 74.93)
-		)
-		(stroke
-			(width 0)
-			(type default)
-		)
-	)
-	(wire
-		(pts
 			(xy 71.12 95.25) (xy 71.12 106.68)
 		)
@@
 	(wire
 		(pts
-			(xy 91.44 77.47) (xy 95.25 77.47)
-		)
-		(stroke
-			(width 0)
-			(type default)
-		)
-	)
-	(wire
-		(pts
 			(xy 142.24 120.65) (xy 142.24 116.84)
 		)
@@
 	)
 	(symbol
-		(lib_name "VCC_3")
-		(lib_id "power:VCC")
-		(at 92.71 74.93 0)
-		(unit 1)
-		(exclude_from_sim no)
-		(in_bom yes)
-		(on_board yes)
-		(dnp no)
-		(property "Reference" "#PWR08"
-			(at 92.71 78.74 0)
-			(effects
-				(font
-					(size 1.27 1.27)
-				)
-				(hide yes)
-			)
-		)
-		(property "Value" "+3.3V"
-			(at 88.9 73.66 0)
-			(effects
-				(font
-					(size 1.27 1.27)
-				)
-			)
-		)
-		(property "Footprint" ""
-			(at 92.71 74.93 0)
-			(effects
-				(font
-					(size 1.27 1.27)
-				)
-				(hide yes)
-			)
-		)
-		(property "Datasheet" ""
-			(at 92.71 74.93 0)
-			(effects
-				(font
-					(size 1.27 1.27)
-				)
-				(hide yes)
-			)
-		)
-		(property "Description" "Power symbol creates a global label with name \"VCC\""
-			(at 92.71 74.93 0)
-			(effects
-				(font
-					(size 1.27 1.27)
-				)
-				(hide yes)
-			)
-		)
-		(pin "1"
-		)
-		(instances
-			(project "Carga util"
-				(path "/afedccfc-6b3f-4582-a9c9-e58b4e8c4739"
-					(reference "#PWR08")
-					(unit 1)
-				)
-			)
-		)
-	)
-	(symbol
 		(lib_id "Connector:Conn_01x04_Pin")
 		(at 97.79 60.96 180)
@@
 	)
 	(symbol
-		(lib_id "Connector:Conn_01x06_Pin")
-		(at 100.33 82.55 180)
+		(lib_id "Connector:Conn_01x04_Pin")
+		(at 100.33 85.09 180)
 		(unit 1)
 		(exclude_from_sim no)
@@
 		(fields_autoplaced yes)
 		(property "Reference" "J3"
-			(at 101.6 80.0099 0)
+			(at 101.6 82.5499 0)
 			(effects
 				(font
@@
 		)
 		(property "Value" "DEBUG"
-			(at 101.6 82.5499 0)
+			(at 101.6 85.0899 0)
 			(effects
 				(font
@@
 		)
 		(property "Footprint" "Connector_PinHeader_2.54mm:PinHeader_1x06_P2.54mm_Vertical"
-			(at 100.33 82.55 0)
+			(at 100.33 85.09 0)
 			(effects
 				(font
@@
 		)
 		(property "Datasheet" "~"
-			(at 100.33 82.55 0)
+			(at 100.33 85.09 0)
 			(effects
 				(font
@@
 			)
 		)
-		(property "Description" "Generic connector, single row, 01x06, script generated"
-			(at 100.33 82.55 0)
+		(property "Description" "Generic connector, single row, 01x04, script generated"
+			(at 100.33 85.09 0)
 			(effects
 				(font
@@
 		(pin "4"
 		)
-		(pin "6"
-		)
-		(pin "5"
-		)
 		(instances
 			(project ""
@@
 					(unit 1)
 				)
-			)
-		)
-	)
-	(symbol
-		(lib_name "GND_4")
-		(lib_id "power:GND")
-		(at 88.9 74.93 0)
-		(unit 1)
-		(exclude_from_sim no)
-		(in_bom yes)
-		(on_board yes)
-		(dnp no)
-		(property "Reference" "#PWR07"
-			(at 88.9 81.28 0)
-			(effects
-				(font
-					(size 1.27 1.27)
-				)
-				(hide yes)
-			)
-		)
-		(property "Value" "GND"
-			(at 86.106 77.724 0)
-			(effects
-				(font
-					(size 1.27 1.27)
-				)
-			)
-		)
-		(property "Footprint" ""
-			(at 88.9 74.93 0)
-			(effects
-				(font
-					(size 1.27 1.27)
-				)
-				(hide yes)
-			)
-		)
-		(property "Datasheet" ""
-			(at 88.9 74.93 0)
-			(effects
-				(font
-					(size 1.27 1.27)
-				)
-				(hide yes)
-			)
-		)
-		(property "Description" "Power symbol creates a global label with name \"GND\" , ground"
-			(at 88.9 74.93 0)
-			(effects
-				(font
-					(size 1.27 1.27)
-				)
-				(hide yes)
-			)
-		)
-		(pin "1"
-		)
-		(instances
-			(project "Carga util"
-				(path "/afedccfc-6b3f-4582-a9c9-e58b4e8c4739"
-					(reference "#PWR07")
-					(unit 1)
-				)
